File: Hardware/EscaramujoLagoMatch.kicad_pcb (KiCad board)
At the start: 2 copper layers, 16 parts, among them J1 Jack_3.5mm_5pin, J2 RJ45, U1 MAX662A

Commit message: Updated footprints
Parts:
- removed RV1: POT, Potentiometers:Potentiometer_Bourns_3296W_3-8Zoll_Inline_ScrewUp
- removed SMA_IN1, SMA_OUT1: SMA_EDGE, sma:SMA
- removed W1, W2: TEST_1P, Measurement_Points:Measurement_Point_Square-TH_Big
- added C10: 100n, Capacitor_SMD:C_0805_2012Metric_Pad1.15x1.40mm_HandSolder, F.Cu at (99.7, 66.8)
- added C11: 100n, Capacitor_SMD:C_0805_2012Metric_Pad1.15x1.40mm_HandSolder, F.Cu at (92.5, 66.8)
- added C12: 10u, Capacitor_THT:C_Disc_D5.0mm_W2.5mm_P2.50mm, F.Cu at (152.4, 67.3)
- added C3: 10uF, Capacitor_THT:C_Disc_D5.0mm_W2.5mm_P2.50mm, F.Cu at (78.8, 80.0)
- added C4: 10uF, Capacitor_THT:C_Disc_D5.0mm_W2.5mm_P2.50mm, F.Cu at (157.5, 49.5)
- added C9: 10uF, Capacitor_THT:C_Disc_D5.0mm_W2.5mm_P2.50mm, F.Cu at (191.8, 59.7)
- added J3: TP_5V, Connector_PinHeader_2.54mm:PinHeader_1x01_P2.54mm_Vertical, F.Cu at (154.9, 26.7)
- added J4: TP_GND, Connector_PinHeader_2.54mm:PinHeader_1x01_P2.54mm_Vertical, F.Cu at (84.8, 47.6)
- added J5: TEMP_PRES, Connector_PinHeader_2.54mm:PinHeader_1x06_P2.54mm_Vertical, F.Cu at (86.4, 21.6)
- added J6: TP_12V, Connector_PinHeader_2.54mm:PinHeader_1x01_P2.54mm_Vertical, F.Cu at (144.8, 26.7)
- added J7: RedPitaya, Connector_PinHeader_2.54mm:PinHeader_2x13_P2.54mm_Vertical, F.Cu at (212.1, 38.1)
- added J8: TP_PMT_CTL_V, Connector_PinHeader_2.54mm:PinHeader_1x01_P2.54mm_Vertical, F.Cu at (79.4, 55.5)
- added R2: 15k, Resistor_THT:R_Axial_DIN0207_L6.3mm_D2.5mm_P10.16mm_Horizontal, F.Cu at (163.8, 24.1)
- added R4: 4k7, Resistor_SMD:R_0805_2012Metric_Pad1.15x1.40mm_HandSolder, F.Cu at (53.7, 62.2)
- added R5: 4k7, Resistor_SMD:R_0805_2012Metric_Pad1.15x1.40mm_HandSolder, F.Cu at (57.5, 62.5)
- added U2: MAX604, Package_DIP:DIP-8_W10.16mm_LongPads, F.Cu at (170.2, 62.2)
- added U3: MAX603, Package_DIP:DIP-8_W10.16mm_LongPads, F.Cu at (170.2, 40.6)
- added U4: MCP41100, Package_DIP:DIP-8_W10.16mm_LongPads, F.Cu at (147.3, 81.3)
- added U5: LM358, Package_DIP:DIP-8_W10.16mm_LongPads, F.Cu at (113.0, 80.0)
- C1, C2: value 1u -> 2u2; footprint Capacitors_ThroughHole:C_Rect_L7_W2.5_P5 -> Capacitor_THT:C_Disc_D5.0mm_W2.5mm_P2.50mm
- C5, C6: footprint Capacitors_ThroughHole:C_Rect_L7_W2.5_P5 -> Capacitor_THT:C_Disc_D5.0mm_W2.5mm_P2.50mm
- C7: value 1n -> 10uF; footprint Capacitors_ThroughHole:C_Rect_L7_W2.5_P5 -> Capacitor_THT:C_Disc_D5.0mm_W2.5mm_P2.50mm
- C8: footprint Capacitors_ThroughHole:C_Rect_L7_W2.5_P5 -> Capacitor_SMD:C_0805_2012Metric_Pad1.15x1.40mm_HandSolder
- J1: value Jack_3.5mm_5pin -> TP_3v3; footprint audioJack5Pin:1503_09 -> Connector_PinHeader_2.54mm:PinHeader_1x01_P2.54mm_Vertical
- J2: footprint Connect:RJ45_8 -> Connector_RJ:RJ45_Amphenol_54602-x08_Horizontal
- R1: value 51 -> 100k; footprint Resistors_ThroughHole:Resistor_Horizontal_RM7mm -> Resistor_SMD:R_0805_2012Metric_Pad1.15x1.40mm_HandSolder
- R3: value 51 -> 18k; footprint Resistors_ThroughHole:Resistor_Horizontal_RM7mm -> Resistor_THT:R_Axial_DIN0207_L6.3mm_D2.5mm_P10.16mm_Horizontal
- U1: footprint Housings_DIP:DIP-8_W7.62mm_LongPads -> Package_DIP:DIP-8_W10.16mm_LongPads
- moved C6 128.7 mm to (190.5, 49.5), turned to 0 degrees
- moved R3 120.9 mm to (163.8, 31.8)
- moved C1 77.1 mm to (141.0, 49.5), turned to 0 degrees
- moved C2 77.0 mm to (141.0, 58.4), turned to 0 degrees
- moved C7 74.3 mm to (124.5, 59.7), turned to 0 degrees
- moved J2 52.1 mm to (121.9, 26.7)
- moved J1 40.0 mm to (81.2, 50.0), turned to 0 degrees
- moved C5 36.5 mm to (121.9, 47.0), turned to 0 degrees
- moved U1 32.8 mm to (68.6, 21.6)
- moved C8 23.0 mm to (106.8, 66.8), turned to 0 degrees
- moved R1 20.7 mm to (50.0, 62.2)
Connections:
- C5 pad 1: VCC -> +5V
- C7 pad 1: Net-(C7-Pad1) -> +3V3
- C7 pad 2: Net-(C7-Pad2) -> GND
- J1 pad 1: GND -> +3V3
- J2 pad 3: Net-(J2-Pad3) -> /PMT_CTRL_V
- J2 pad 5: VCC -> +5V
- R1 pad 1: Net-(R1-Pad1) -> Net-(C12-Pad1)
- R1 pad 2: GND -> /PMT_CTRL_V_NF
- R3 pad 1: Net-(R1-Pad1) -> Net-(R2-Pad1)
- R3 pad 2: Net-(C7-Pad1) -> Net-(R3-Pad2)
- U1 pad 5: VCC -> +5V
Routing:
- net GND: track 239.1 -> 0.00 mm, vias 2 -> 0
- net VCC: track 97.1 -> 0.00 mm
- net /12V: track 47.4 -> 0.00 mm
- net Net-(J2-Pad3): track 30.6 -> 0.00 mm
- net Net-(R1-Pad1): track 22.5 -> 0.00 mm
- net Net-(C7-Pad2): track 19.0 -> 0.00 mm
- net Net-(C1-Pad2): track 8.71 -> 0.00 mm
- net Net-(C2-Pad2): track 8.42 -> 0.00 mm
- net Net-(C1-Pad1): track 7.69 -> 0.00 mm
- net Net-(C2-Pad1): track 7.60 -> 0.00 mm
- net Net-(C7-Pad1): track 6.37 -> 0.00 mm
- removed copper zone on B.Cu, net GND
Other:
- board text removed: "+5 VDC"
- board text removed: "LAGO + Escaramujo"
- board text removed: "OUT"
- board text removed: "PMT IN"

Commit message: PCB Finished
Parts:
- added J10: I2C, Connector_PinHeader_2.54mm:PinHeader_1x04_P2.54mm_Vertical, F.Cu at (68.6, 180.6)
- added J9: TP_GND, Connector_PinHeader_2.54mm:PinHeader_1x01_P2.54mm_Vertical, F.Cu at (100.3, 170.2)
- C10, C11, C8, R1, R4, R5: moved to B.Cu
- moved J7 206.2 mm to (26.7, 128.3)
- moved C6 162.0 mm to (62.2, 148.6), turned to 90 degrees
- moved R3 157.3 mm to (64.5, 153.7), turned to 270 degrees
- moved J5 151.1 mm to (78.2, 172.5), turned to 270 degrees
- moved U3 149.7 mm to (47.0, 125.7)
- moved R2 149.3 mm to (81.3, 148.6)
- moved C4 142.7 mm to (41.9, 133.3), turned to 90 degrees
- moved C9 139.2 mm to (68.6, 124.5), turned to 270 degrees
- moved C1 138.3 mm to (41.9, 146.1), turned to 90 degrees
- moved C2 134.0 mm to (41.9, 148.6), turned to 270 degrees
- moved U4 126.8 mm to (47.0, 158.8)
- moved J2 126.1 mm to (101.6, 151.1), turned to 90 degrees
- moved R4 124.5 mm to (73.2, 185.2), turned to 90 degrees
- moved U1 123.8 mm to (47.0, 143.5)
- moved R5 123.3 mm to (70.6, 185.2), turned to 90 degrees
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Connections:
- J7 pad 11: /SPI_CS -> (no net)
- J7 pad 14: /5V_UNREG -> (no net)
- J7 pad 15: /SPI_MOSI -> GND
- J7 pad 16: /SPI_CLK -> GND
- J7 pad 17: (no net) -> /I2C_SDA
- J7 pad 19: GND -> (no net)
- J7 pad 21: (no net) -> /SPI_CS
- J7 pad 22: (no net) -> /SPI_CLK
- J7 pad 24: (no net) -> /SPI_MOSI
- J7 pad 26: (no net) -> /5V_UNREG
- J7 pad 8: GND -> (no net)
- J7 pad 9: /I2C_SDA -> (no net)
- U5 pad 4: (no net) -> GND
- U5 pad 8: (no net) -> +3V3
Routing:
- net GND: track 0.00 -> 368.9 mm, vias 0 -> 2
- net +3V3: track 0.00 -> 233.9 mm, vias 0 -> 6
- net +5V: track 0.00 -> 120.0 mm, vias 0 -> 2
- net /I2C_SDA: track 0.00 -> 88.3 mm
- net /I2C_SCL: track 0.00 -> 80.5 mm, vias 0 -> 2
- net /5V_UNREG: track 0.00 -> 64.2 mm, vias 0 -> 2
- net /12V: track 0.00 -> 57.2 mm, vias 0 -> 2
- net /PMT_CTRL_V: track 0.00 -> 44.0 mm
- net /SPI_CS: track 0.00 -> 42.7 mm, vias 0 -> 2
- net Net-(R3-Pad2): track 0.00 -> 30.7 mm
- net Net-(C12-Pad1): track 0.00 -> 26.4 mm
- net /SPI_MOSI: track 0.00 -> 20.9 mm
- net /SPI_CLK: track 0.00 -> 20.9 mm
- net Net-(R2-Pad1): track 0.00 -> 18.9 mm
- net /PMT_CTRL_V_NF: track 0.00 -> 6.35 mm
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- added copper zone on B.Cu, net GND
Other:
- board outline added: 113 x 80 mm
- net class Default: trace_width 0.4 -> 0.75; via_dia 1.4 -> 2
- board text added: "12V"
- board text added: "3v3"
- board text added: "5V"
- board text added: "GND"
- board text added: "Vctrl PMT"
