File: Hardware/EscaramujoLagoMatch.kicad_pcb (KiCad board)
At the start: 2 copper layers, 16 parts, among them J1 Jack_3.5mm_5pin, J2 RJ45, U1 MAX662A

Commit message: Add files via upload
Parts:
- removed RV1: POT, Potentiometers:Potentiometer_Bourns_3296W_3-8Zoll_Inline_ScrewUp
- removed SMA_IN1, SMA_OUT1: SMA_EDGE, sma:SMA
- removed W1, W2: TEST_1P, Measurement_Points:Measurement_Point_Square-TH_Big
- added C10: 100n, Capacitor_SMD:C_0805_2012Metric_Pad1.15x1.40mm_HandSolder, B.Cu at (97.8, 127.2)
- added C11: 100n, Capacitor_SMD:C_0805_2012Metric_Pad1.15x1.40mm_HandSolder, B.Cu at (63.5, 126.0)
- added C12: 10u, Capacitor_THT:C_Disc_D5.0mm_W2.5mm_P2.50mm, F.Cu at (81.3, 153.7)
- added C3: 10uF, Capacitor_THT:C_Disc_D5.0mm_W2.5mm_P2.50mm, F.Cu at (67.3, 135.9)
- added C4: 10uF, Capacitor_THT:C_Disc_D5.0mm_W2.5mm_P2.50mm, F.Cu at (41.9, 133.3)
- added C9: 10uF, Capacitor_THT:C_Disc_D5.0mm_W2.5mm_P2.50mm, F.Cu at (68.6, 124.5)
- added J10: I2C, Connector_PinHeader_2.54mm:PinHeader_1x04_P2.54mm_Vertical, F.Cu at (68.6, 180.6)
- added J3: TP_5V, Connector_PinHeader_2.54mm:PinHeader_1x01_P2.54mm_Vertical, F.Cu at (101.6, 134.6)
- added J4: TP_GND, Connector_PinHeader_2.54mm:PinHeader_1x01_P2.54mm_Vertical, F.Cu at (114.3, 134.6)
- added J5: TEMP_PRES, Connector_PinHeader_2.54mm:PinHeader_1x06_P2.54mm_Vertical, F.Cu at (78.2, 172.5)
- added J6: TP_12V, Connector_PinHeader_2.54mm:PinHeader_1x01_P2.54mm_Vertical, F.Cu at (95.2, 134.6)
- added J7: RedPitaya, Connector_PinHeader_2.54mm:PinHeader_2x13_P2.54mm_Vertical, F.Cu at (26.7, 128.3)
- added J8: TP_PMT_CTL_V, Connector_PinHeader_2.54mm:PinHeader_1x01_P2.54mm_Vertical, F.Cu at (100.3, 162.6)
- added J9: TP_GND, Connector_PinHeader_2.54mm:PinHeader_1x01_P2.54mm_Vertical, F.Cu at (100.3, 170.2)
- added R2: 15k, Resistor_THT:R_Axial_DIN0207_L6.3mm_D2.5mm_P10.16mm_Horizontal, F.Cu at (81.3, 148.6)
- added R4: 4k7, Resistor_SMD:R_0805_2012Metric_Pad1.15x1.40mm_HandSolder, B.Cu at (73.2, 185.2)
- added R5: 4k7, Resistor_SMD:R_0805_2012Metric_Pad1.15x1.40mm_HandSolder, B.Cu at (70.6, 185.2)
- added U2: MAX604, Package_DIP:DIP-8_W10.16mm_LongPads, F.Cu at (74.9, 125.7)
- added U3: MAX603, Package_DIP:DIP-8_W10.16mm_LongPads, F.Cu at (47.0, 125.7)
- added U4: MCP41100, Package_DIP:DIP-8_W10.16mm_LongPads, F.Cu at (47.0, 158.8)
- added U5: LM358, Package_DIP:DIP-8_W10.16mm_LongPads, F.Cu at (83.8, 160.0)
- C1, C2: value 1u -> 2u2; footprint Capacitors_ThroughHole:C_Rect_L7_W2.5_P5 -> Capacitor_THT:C_Disc_D5.0mm_W2.5mm_P2.50mm
- C5, C6: footprint Capacitors_ThroughHole:C_Rect_L7_W2.5_P5 -> Capacitor_THT:C_Disc_D5.0mm_W2.5mm_P2.50mm
- C7: value 1n -> 10uF; footprint Capacitors_ThroughHole:C_Rect_L7_W2.5_P5 -> Capacitor_THT:C_Disc_D5.0mm_W2.5mm_P2.50mm
- C8: footprint Capacitors_ThroughHole:C_Rect_L7_W2.5_P5 -> Capacitor_SMD:C_0805_2012Metric_Pad1.15x1.40mm_HandSolder; moved to B.Cu
- J1: value Jack_3.5mm_5pin -> TP_3v3; footprint audioJack5Pin:1503_09 -> Connector_PinHeader_2.54mm:PinHeader_1x01_P2.54mm_Vertical
- J2: footprint Connect:RJ45_8 -> Connector_RJ:RJ45_Amphenol_54602-x08_Horizontal
- R1: value 51 -> 100k; footprint Resistors_ThroughHole:Resistor_Horizontal_RM7mm -> Resistor_SMD:R_0805_2012Metric_Pad1.15x1.40mm_HandSolder; moved to B.Cu
- R3: value 51 -> 18k; footprint Resistors_ThroughHole:Resistor_Horizontal_RM7mm -> Resistor_THT:R_Axial_DIN0207_L6.3mm_D2.5mm_P10.16mm_Horizontal
- U1: footprint Housings_DIP:DIP-8_W7.62mm_LongPads -> Package_DIP:DIP-8_W10.16mm_LongPads
- moved J2 130.3 mm to (101.6, 151.1), turned to 90 degrees
- moved R1 122.0 mm to (80.0, 159.0), turned to 270 degrees
- moved R3 107.6 mm to (64.5, 153.7), turned to 270 degrees
- moved C6 106.2 mm to (62.2, 148.6), turned to 90 degrees
- moved C1 92.7 mm to (41.9, 146.1)
- moved U1 92.6 mm to (47.0, 143.5)
- moved C2 92.2 mm to (41.9, 148.6)
- moved C8 90.0 mm to (67.3, 147.6)
- moved J1 82.9 mm to (108.0, 134.6), turned to 0 degrees
- moved C7 82.8 mm to (91.4, 125.8), turned to 270 degrees
- moved C5 78.5 mm to (78.8, 139.7), turned to 0 degrees
Connections:
- C5 pad 1: VCC -> +5V
- C7 pad 1: Net-(C7-Pad1) -> +3V3
- C7 pad 2: Net-(C7-Pad2) -> GND
- J1 pad 1: GND -> +3V3
- J2 pad 3: Net-(J2-Pad3) -> /PMT_CTRL_V
- J2 pad 5: VCC -> +5V
- R1 pad 1: Net-(R1-Pad1) -> Net-(C12-Pad1)
- R1 pad 2: GND -> /PMT_CTRL_V_NF
- R3 pad 1: Net-(R1-Pad1) -> Net-(R2-Pad1)
- R3 pad 2: Net-(C7-Pad1) -> Net-(R3-Pad2)
- U1 pad 5: VCC -> +5V
Routing:
- net +3V3: track 0.00 -> 233.9 mm, vias 0 -> 6
- net GND: track 239.1 -> 368.9 mm
- net +5V: track 0.00 -> 120.0 mm, vias 0 -> 2
- net VCC: track 97.1 -> 0.00 mm
- net /I2C_SDA: track 0.00 -> 88.3 mm
- net /I2C_SCL: track 0.00 -> 80.5 mm, vias 0 -> 2
- net /5V_UNREG: track 0.00 -> 64.2 mm, vias 0 -> 2
- net /PMT_CTRL_V: track 0.00 -> 44.0 mm
- net /SPI_CS: track 0.00 -> 42.7 mm, vias 0 -> 2
- net Net-(R3-Pad2): track 0.00 -> 30.7 mm
- net Net-(J2-Pad3): track 30.6 -> 0.00 mm
- net Net-(C12-Pad1): track 0.00 -> 26.4 mm
- net Net-(R1-Pad1): track 22.5 -> 0.00 mm
- net /SPI_MOSI: track 0.00 -> 20.9 mm
- net /SPI_CLK: track 0.00 -> 20.9 mm
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Other:
- board outline added: 113 x 80 mm
- net class Default: trace_width 0.4 -> 0.75; via_dia 1.4 -> 2
- board text added: "12V"
- board text added: "3v3"
- board text added: "5V"
- board text added: "GND"
- board text added: "Vctrl PMT"
- board text removed: "+5 VDC"
- board text removed: "LAGO + Escaramujo"
- board text removed: "OUT"
- board text removed: "PMT IN"

Commit message: Add files via upload
Parts:
- removed R5: 4k7, Resistor_SMD:R_0805_2012Metric_Pad1.15x1.40mm_HandSolder
- added C13: 100n, Capacitor_SMD:C_0805_2012Metric_Pad1.15x1.40mm_HandSolder, B.Cu at (87.5, 120.0)
- added C14: 10u, Capacitor_THT:C_Disc_D5.0mm_W2.5mm_P2.50mm, F.Cu at (90.5, 118.4)
- added C15: 100n, Capacitor_SMD:C_0805_2012Metric_Pad1.15x1.40mm_HandSolder, B.Cu at (46.5, 103.5)
- added D1: LED, LED_THT:LED_D5.0mm, F.Cu at (82.7, 87.5)
- J5: value TEMP_PRES -> Sensor; footprint Connector_PinHeader_2.54mm:PinHeader_1x06_P2.54mm_Vertical -> Connector_PinHeader_2.54mm:PinHeader_1x04_P2.54mm_Vertical
- R2: value 15k -> 5.1k
- R3: value 18k -> 3k
- R4: value 4k7 -> 330; footprint Resistor_SMD:R_0805_2012Metric_Pad1.15x1.40mm_HandSolder -> Resistor_THT:R_Axial_DIN0207_L6.3mm_D2.5mm_P10.16mm_Horizontal; moved to F.Cu
- U1, U2, U3, U5: footprint Package_DIP:DIP-8_W10.16mm_LongPads -> Package_DIP:DIP-8_W7.62mm_Socket
- U4: value MCP41100 -> TLV5616CD; footprint Package_DIP:DIP-8_W10.16mm_LongPads -> SOIC127P600X175-8N; moved to B.Cu
- moved J10 108.1 mm to (121.0, 86.0), turned to 0 degrees
- moved R4 97.7 mm to (74.0, 87.5), turned to 180 degrees
- moved J5 94.5 mm to (116.0, 85.9), turned to 0 degrees
- moved J7 93.5 mm to (116.5, 102.2)
- moved J8 89.4 mm to (36.5, 100.0)
- moved J4 77.5 mm to (45.0, 100.0)
- moved J9 73.9 mm to (36.5, 133.0)
- moved J2 70.0 mm to (45.8, 108.8), turned to 270 degrees
- moved U4 65.7 mm to (99.6, 119.4), turned to 180 degrees
- moved J3 65.6 mm to (36.5, 126.5)
- moved U5 65.0 mm to (92.0, 95.5)
- moved J1 63.0 mm to (45.0, 133.0)
- moved R1 55.0 mm to (96.5, 106.5), turned to 180 degrees
- moved J6 50.9 mm to (45.0, 126.5)
- moved C12 48.1 mm to (88.0, 106.0), turned to 90 degrees
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Connections:
- J10 pad 2: /I2C_SDA -> GND
- J10 pad 4: GND -> /I2C_SDA
- J2 pad 1: (no net) -> Net-(J2-Pad1)
- J2 pad 2: (no net) -> Net-(J2-Pad2)
- J2 pad 7: (no net) -> Net-(J2-Pad7)
- J2 pad 8: (no net) -> Net-(J2-Pad8)
- J5 pad 1: /I2C_SCL -> +3V3
- J5 pad 2: (no net) -> GND
- J5 pad 3: /I2C_SDA -> /I2C_SCL
- J5 pad 4: (no net) -> /I2C_SDA
- J7 pad 1: (no net) -> Net-(J7-Pad1)
- J7 pad 10: (no net) -> Net-(J7-Pad10)
- J7 pad 11: (no net) -> Net-(J7-Pad11)
- J7 pad 12: (no net) -> Net-(J7-Pad12)
- J7 pad 13: (no net) -> Net-(J7-Pad13)
- J7 pad 14: (no net) -> Net-(J7-Pad14)
- J7 pad 19: (no net) -> Net-(J7-Pad19)
- J7 pad 2: (no net) -> Net-(J7-Pad2)
- J7 pad 20: (no net) -> Net-(J7-Pad20)
- J7 pad 23: (no net) -> Net-(J7-Pad23)
- J7 pad 25: (no net) -> Net-(J7-Pad25)
- J7 pad 3: (no net) -> Net-(J7-Pad3)
- J7 pad 4: (no net) -> Net-(J7-Pad4)
- J7 pad 5: (no net) -> Net-(J7-Pad5)
- J7 pad 6: (no net) -> Net-(J7-Pad6)
- J7 pad 7: (no net) -> Net-(J7-Pad7)
- J7 pad 8: (no net) -> Net-(J7-Pad8)
- J7 pad 9: (no net) -> Net-(J7-Pad9)
- R2 pad 1: Net-(R2-Pad1) -> +3V3
- R2 pad 2: +3V3 -> Net-(R2-Pad2)
- R3 pad 1: Net-(R2-Pad1) -> Net-(R2-Pad2)
- R3 pad 2: Net-(R3-Pad2) -> GND
- R4 pad 1: +3V3 -> Net-(D1-Pad1)
- R4 pad 2: /I2C_SCL -> GND
- U4 pad 1: /SPI_CS -> /SPI_MOSI
- U4 pad 3: /SPI_MOSI -> GND
- U4 pad 4: GND -> /SPI_CS
- U4 pad 5: Net-(R3-Pad2) -> GND
- U4 pad 6: Net-(R3-Pad2) -> Net-(R2-Pad2)
- U4 pad 7: GND -> Net-(U4-Pad7)
- U5 pad 3: Net-(R3-Pad2) -> Net-(U4-Pad7)
Routing:
- net /5V_UNREG: track 64.2 -> 192.7 mm, vias 2 -> 4
- net +3V3: track 233.9 -> 154.3 mm, vias 6 -> 0
- net /PMT_CTRL_V: track 44.0 -> 100.7 mm
- net /I2C_SDA: track 88.3 -> 38.0 mm
- net +5V: track 120.0 -> 167.9 mm
- net /I2C_SCL: track 80.5 -> 41.4 mm, vias 2 -> 0
- net Net-(R3-Pad2): track 30.7 -> 0.00 mm
- net /SPI_CLK: track 20.9 -> 47.0 mm
- net /12V: track 57.2 -> 82.9 mm, vias 2 -> 0
- net Net-(U4-Pad7): track 0.00 -> 24.5 mm, vias 0 -> 2
- net /SPI_MOSI: track 20.9 -> 42.6 mm
- net Net-(R2-Pad1): track 18.9 -> 0.00 mm
- net Net-(R2-Pad2): track 0.00 -> 15.9 mm
- net /SPI_CS: track 42.7 -> 27.9 mm
- net Net-(C12-Pad1): track 26.4 -> 15.8 mm
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Other:
- board size 113 x 80 mm -> 97 x 60.5 mm
- net class Default: clearance 0.2 -> 0.6; trace_width 0.75 -> 0.6; via_dia 2 -> 1.2
- rule pad_to_mask_clearance: 0.2 -> 0
- rule trace_clearance: 0.2 -> 0.6
- rule trace_min: 0.4 -> 0.2
- rule via_min_drill: 0.4 -> 0.3
- rule via_min_size: 0.8 -> 0.4
- board text added: "3.3V"
- board text added: "ECFM - LAGO"
- board text added: "RED PITAYA"
- board text added: "VPMT"
- board text removed: "3v3"
- board text removed: "Vctrl PMT"
