File: Hardware/EscaramujoLagoMatch.sch (KiCad schematic (older format))
At the start: 8 parts

Commit message: PCB Design Done
Includes custom library files
Parts:
- removed C?: C, symbol C
- removed C?: CP, symbol CP
- removed J?: JACK_TRS_6PINS, symbol JACK_TRS_6PINS
- removed R?: R, symbol R
- added C1, C2: 1u, Capacitors_ThroughHole:C_Rect_L7_W2.5_P5, symbol CP
- added C5, C6: 10u, Capacitors_ThroughHole:C_Rect_L7_W2.5_P5, symbol CP
- added C7: 1n, Capacitors_ThroughHole:C_Rect_L7_W2.5_P5, symbol C
- added C8: 100n, Capacitors_ThroughHole:C_Rect_L7_W2.5_P5, symbol C
- added J1: Jack_3.5mm_5pin, audioJack5Pin:1503_09, symbol Jack_3.5mm_5pin
- added R1, R3: 51, Resistors_ThroughHole:Resistor_Horizontal_RM7mm, symbol R
- added RV1: POT, Potentiometers:Potentiometer_Bourns_3296W_3-8Zoll_Inline_ScrewUp, symbol POT
- added W1, W2: TEST_1P, Measurement_Points:Measurement_Point_Square-TH_Big, symbol TEST_1P
- J2: renamed from J?; footprint (none) -> Connect:RJ45_8
- SMA_IN1: renamed from SMA_IN; footprint (none) -> sma:SMA
- SMA_OUT1: renamed from SMA_OUT; footprint (none) -> sma:SMA
- U1: renamed from U?; footprint (none) -> Housings_DIP:DIP-8_W7.62mm_LongPads
Connections:
- net labels added: 12V, VCC
- wire segments 0 -> 58
- no-connect marks 0 -> 8
Other:
- moved on the sheet: SMA_IN1, SMA_OUT1

Commit message: Updated footprints
Parts:
- removed C7: 1n, Capacitors_ThroughHole:C_Rect_L7_W2.5_P5, symbol C
- removed J1: Jack_3.5mm_5pin, audioJack5Pin:1503_09, symbol Jack_3.5mm_5pin
- removed R1, R3: 51, Resistors_ThroughHole:Resistor_Horizontal_RM7mm, symbol R
- removed RV1: POT, Potentiometers:Potentiometer_Bourns_3296W_3-8Zoll_Inline_ScrewUp, symbol POT
- removed SMA_IN1, SMA_OUT1: SMA_EDGE, sma:SMA, symbol SMA_EDGE
- removed W1, W2: TEST_1P, Measurement_Points:Measurement_Point_Square-TH_Big, symbol TEST_1P
- added C10, C11: 100n, Capacitor_SMD:C_0805_2012Metric_Pad1.15x1.40mm_HandSolder, symbol Device:C
- added C12: 10u, Capacitor_THT:C_Disc_D5.0mm_W2.5mm_P2.50mm, symbol Device:CP
- added C3, C4, C7, C9: 10uF, Capacitor_THT:C_Disc_D5.0mm_W2.5mm_P2.50mm, symbol Device:CP
- added J1: TP_3v3, Connector_PinHeader_2.54mm:PinHeader_1x01_P2.54mm_Vertical, symbol Connector_Generic:Conn_01x01
- added J3: TP_5V, Connector_PinHeader_2.54mm:PinHeader_1x01_P2.54mm_Vertical, symbol Connector_Generic:Conn_01x01
- added J4: TP_GND, Connector_PinHeader_2.54mm:PinHeader_1x01_P2.54mm_Vertical, symbol Connector_Generic:Conn_01x01
- added J5: TEMP_PRES, Connector_PinHeader_2.54mm:PinHeader_1x06_P2.54mm_Vertical, symbol Connector_Generic:Conn_01x06
- added J6: TP_12V, Connector_PinHeader_2.54mm:PinHeader_1x01_P2.54mm_Vertical, symbol Connector_Generic:Conn_01x01
- added J7: RedPitaya, Connector_PinHeader_2.54mm:PinHeader_2x13_P2.54mm_Vertical, symbol Connector_Generic:Conn_02x13_Counter_Clockwise
- added J8: TP_PMT_CTL_V, Connector_PinHeader_2.54mm:PinHeader_1x01_P2.54mm_Vertical, symbol Connector_Generic:Conn_01x01
- added R1: 100k, Resistor_SMD:R_0805_2012Metric_Pad1.15x1.40mm_HandSolder, symbol Device:R
- added R2: 15k, Resistor_THT:R_Axial_DIN0207_L6.3mm_D2.5mm_P10.16mm_Horizontal, symbol Device:R
- added R3: 18k, Resistor_THT:R_Axial_DIN0207_L6.3mm_D2.5mm_P10.16mm_Horizontal, symbol Device:R
- added R4, R5: 4k7, Resistor_SMD:R_0805_2012Metric_Pad1.15x1.40mm_HandSolder, symbol Device:R
- added U2: MAX604, Package_DIP:DIP-8_W10.16mm_LongPads, symbol Regulator_Linear:MAX604
- added U3: MAX603, Package_DIP:DIP-8_W10.16mm_LongPads, symbol Regulator_Linear:MAX603
- added U4: MCP41100, Package_DIP:DIP-8_W10.16mm_LongPads, symbol Potentiometer_Digital:MCP41100
- added U5: LM358, Package_DIP:DIP-8_W10.16mm_LongPads, symbol Amplifier_Operational:LM358
- C1, C2: value 1u -> 2u2; footprint Capacitors_ThroughHole:C_Rect_L7_W2.5_P5 -> Capacitor_THT:C_Disc_D5.0mm_W2.5mm_P2.50mm; symbol CP -> Device:CP
- C5, C6: footprint Capacitors_ThroughHole:C_Rect_L7_W2.5_P5 -> Capacitor_THT:C_Disc_D5.0mm_W2.5mm_P2.50mm; symbol CP -> Device:CP
- C8: footprint Capacitors_ThroughHole:C_Rect_L7_W2.5_P5 -> Capacitor_SMD:C_0805_2012Metric_Pad1.15x1.40mm_HandSolder; symbol C -> Device:C
- J2: footprint Connect:RJ45_8 -> Connector_RJ:RJ45_Amphenol_54602-x08_Horizontal; symbol RJ45 -> EscaramujoLagoMatch-rescue:RJ45
- U1: footprint Housings_DIP:DIP-8_W7.62mm_LongPads -> Package_DIP:DIP-8_W10.16mm_LongPads; symbol MAX662A -> ProjectSpecificParts:MAX662A
Connections:
- net 12V: now also J6.1 (Pin_1)
- net GND: now also C10.2, C11.2, C12.2, C3.2, C4.2, C7.2, C9.2, J4.1 (Pin_1), J5.5 (Pin_5), J7.19 (Pin_19), J7.8 (Pin_8), U2.2 (GND), U2.3 (GND), U2.5 (SET), U2.6 (GND), U2.7 (GND), U3.2 (GND), U3.3 (GND), U3.5 (SET), U3.6 (GND), U3.7 (GND), U4.4 (VSS), U4.7 (PB0)
- net PMT_CTRL_V: now reaches J2.3
- net PMT_CTRL_V: now also J8.1 (Pin_1), U5.6 (-), U5.7
- net VCC renamed +5V
- net +5V: now also C11.1, C3.1, C9.1, J3.1 (Pin_1), U2.1 (IN), U2.4 (~OFF), U3.8 (OUT)
- new net: R3.2, U4.5 (PA0), U4.6 (PW0), U5.3 (+)
- new net: R2.1, R3.1
- new net: C12.1, R1.1, U5.5 (+)
- new net +3V3: C10.1, C7.1, J1.1 (Pin_1), J5.6 (Pin_6), R2.2, R4.1, R5.1, U2.8 (OUT), U4.8 (VDD)
- new net 5V_UNREG: C4.1, J7.14 (Pin_14), U3.1 (IN), U3.4 (~OFF)
- new net I2C_SCL: J5.1 (Pin_1), J7.18 (Pin_18), R4.2
- new net I2C_SDA: J5.3 (Pin_3), J7.9 (Pin_9), R5.2
- new net PMT_CTRL_V_NF: R1.2, U5.1, U5.2 (-)
- new net SPI_CLK: J7.16 (Pin_16), U4.2 (SCK)
- new net SPI_CS: J7.11 (Pin_11), U4.1 (~CS)
- new net SPI_MOSI: J7.15 (Pin_15), U4.3 (SI)
- no-connect marks 8 -> 25

Commit message: PCB Finished
Parts:
- added J10: I2C, Connector_PinHeader_2.54mm:PinHeader_1x04_P2.54mm_Vertical, symbol Connector_Generic:Conn_01x04
- added J9: TP_GND, Connector_PinHeader_2.54mm:PinHeader_1x01_P2.54mm_Vertical, symbol Connector_Generic:Conn_01x01
- added unit 3 of U5
Connections:
- net +3V3: now also J10.1 (Pin_1), U5.8 (V+)
- net 5V_UNREG: now also J7.26 (Pin_26); no longer J7.14 (Pin_14)
- net GND: now also J7.15 (Pin_15), J7.16 (Pin_16), J10.4 (Pin_4), J9.1 (Pin_1), U5.4 (V-); no longer J7.19 (Pin_19), J7.8 (Pin_8)
- net I2C_SCL: now also J10.3 (Pin_3)
- net I2C_SDA: now also J7.17 (Pin_17), J10.2 (Pin_2); no longer J7.9 (Pin_9)
- net SPI_CLK: now also J7.22 (Pin_22); no longer J7.16 (Pin_16)
- net SPI_CS: now also J7.21 (Pin_21); no longer J7.11 (Pin_11)
- net SPI_MOSI: now also J7.24 (Pin_24); no longer J7.15 (Pin_15)
Changed lines of the file:
@@
 L power:GND #PWR017
 U 1 1 5C539110
-P 7950 2950
-F 0 "#PWR017" H 7950 2700 50  0001 C CNN
-F 1 "GND" V 7955 2822 50  0000 R CNN
-F 2 "" H 7950 2950 50  0001 C CNN
-F 3 "" H 7950 2950 50  0001 C CNN
-	1    7950 2950
-	0    -1   -1   0
-$EndComp
-Wire Wire Line
-	7950 2950 7800 2950
-Wire Wire Line
-	7800 3450 7950 3450
-$Comp
-L power:GND #PWR016
-U 1 1 5C53AF16
-P 7150 2950
-F 0 "#PWR016" H 7150 2700 50  0001 C CNN
-F 1 "GND" V 7155 2822 50  0000 R CNN
-F 2 "" H 7150 2950 50  0001 C CNN
-F 3 "" H 7150 2950 50  0001 C CNN
-	1    7150 2950
-	0    1    1    0
-$EndComp
-Wire Wire Line
-	7300 2950 7150 2950
-Wire Wire Line
-	7300 3050 6500 3050
-Text Label 6500 3050 0    50   ~ 0
+P 8000 3550
+F 0 "#PWR017" H 8000 3300 50  0001 C CNN
+F 1 "GND" V 8005 3422 50  0000 R CNN
+F 2 "" H 8000 3550 50  0001 C CNN
+F 3 "" H 8000 3550 50  0001 C CNN
+	1    8000 3550
+	1    0    0    -1
+$EndComp
+Text Label 8300 3150 2    50   ~ 0
 I2C_SDA
-Wire Wire Line
-	7800 3050 8500 3050
-Text Label 8500 3050 2    50   ~ 0
+Text Label 8300 3050 2    50   ~ 0
 I2C_SCL
-Wire Wire Line
-	7800 3250 8500 3250
-Wire Wire Line
-	7800 3350 8500 3350
-Wire Wire Line
-	7300 3250 6500 3250
-Text Label 8500 3250 2    50   ~ 0
+Text Label 8300 2650 2    50   ~ 0
 SPI_CLK
-Text Label 8500 3350 2    50   ~ 0
+Text Label 8300 2450 2    50   ~ 0
 SPI_MOSI
-Text Label 6500 3250 0    50   ~ 0
+Text Label 8300 2750 2    50   ~ 0
 SPI_CS
-Text Label 7950 3450 0    50   ~ 0
+Text Label 8300 2250 2    50   ~ 0
 5V_UNREG
 $Comp
@@
 	2650 1250 2500 1250
 Connection ~ 2500 1250
-NoConn ~ 7800 3150
 NoConn ~ 7300 3150
 NoConn ~ 7300 3350
 NoConn ~ 7300 3450
 NoConn ~ 7300 2850
-NoConn ~ 7800 2850
-NoConn ~ 7800 2750
-NoConn ~ 7800 2650
-NoConn ~ 7800 2550
-NoConn ~ 7800 2450
-NoConn ~ 7800 2350
 NoConn ~ 7300 2350
 NoConn ~ 7300 2450
@@
 NoConn ~ 7300 2650
 NoConn ~ 7300 2750
-NoConn ~ 7800 2250
 NoConn ~ 7300 2250
 NoConn ~ 5750 1500
@@
 Wire Wire Line
 	3400 4800 3300 4800
+Wire Wire Line
+	8000 3550 8000 3350
+Wire Wire Line
+	8000 3250 7800 3250
+Wire Wire Line
+	7800 3350 8000 3350
+Connection ~ 8000 3350
+Wire Wire Line
+	8000 3350 8000 3250
+Wire Wire Line
+	7800 3150 8300 3150
+Wire Wire Line
+	7800 3050 8300 3050
+NoConn ~ 7300 3250
+NoConn ~ 7300 2950
+NoConn ~ 7300 3050
+Wire Wire Line
+	7800 2750 8300 2750
+Wire Wire Line
+	7800 2650 8300 2650
+Wire Wire Line
+	7800 2450 8300 2450
+Wire Wire Line
+	7800 2250 8300 2250
+NoConn ~ 7800 2350
+NoConn ~ 7800 3450
+$Comp
+L Connector_Generic:Conn_01x04 J10
+U 1 1 5C896E99
+P 9150 1300
+F 0 "J10" H 9230 1292 50  0000 L CNN
+F 1 "I2C" H 9230 1201 50  0000 L CNN
+F 2 "Connector_PinHeader_2.54mm:PinHeader_1x04_P2.54mm_Vertical" H 9150 1300 50  0001 C CNN
+F 3 "~" H 9150 1300 50  0001 C CNN
+	1    9150 1300
+	1    0    0    -1
+$EndComp
+Wire Wire Line
+	8950 1300 8300 1300
+Wire Wire Line
+	8950 1400 8300 1400
+$Comp
+L power:GND #PWR023
+U 1 1 5C897059
+P 8750 1600
+F 0 "#PWR023" H 8750 1350 50  0001 C CNN
+F 1 "GND" H 8755 1427 50  0000 C CNN
+F 2 "" H 8750 1600 50  0001 C CNN
+F 3 "" H 8750 1600 50  0001 C CNN
+	1    8750 1600
+	1    0    0    -1
+$EndComp
+Wire Wire Line
+	8950 1500 8750 1500
+Wire Wire Line
+	8750 1500 8750 1600
+$Comp
+L power:+3V3 #PWR022
+U 1 1 5C89706B
+P 8600 1050
+F 0 "#PWR022" H 8600 900 50  0001 C CNN
+F 1 "+3V3" H 8615 1223 50  0000 C CNN
+F 2 "" H 8600 1050 50  0001 C CNN
+F 3 "" H 8600 1050 50  0001 C CNN
+	1    8600 1050
+	1    0    0    -1
+$EndComp
+Wire Wire Line
+	8950 1200 8600 1200
+Wire Wire Line
+	8600 1200 8600 1050
+Text Label 8300 1300 0    50   ~ 0
+I2C_SDA
+Text Label 8300 1400 0    50   ~ 0
+I2C_SCL
+NoConn ~ 7800 2550
+$Comp
+L Amplifier_Operational:LM358 U5
+U 3 1 5C8ADF24
+P 10550 3450
+F 0 "U5" H 10508 3496 50  0000 L CNN
+F 1 "LM358" H 10508 3405 50  0000 L CNN
+F 2 "Package_DIP:DIP-8_W10.16mm_LongPads" H 10550 3450 50  0001 C CNN
+F 3 "http://www.ti.com/lit/ds/symlink/lm2904-n.pdf" H 10550 3450 50  0001 C CNN
+	3    10550 3450
+	1    0    0    -1
+$EndComp
+$Comp
+L power:GND #PWR0102
+U 1 1 5C8AE0B0
+P 10450 3850
+F 0 "#PWR0102" H 10450 3600 50  0001 C CNN
+F 1 "GND" H 10455 3677 50  0000 C CNN
+F 2 "" H 10450 3850 50  0001 C CNN
+F 3 "" H 10450 3850 50  0001 C CNN
+	1    10450 3850
+	1    0    0    -1
+$EndComp
+Wire Wire Line
+	10450 3850 10450 3750
+$Comp
+L power:+3V3 #PWR0103
+U 1 1 5C8B4D2A
+P 10450 3050
+F 0 "#PWR0103" H 10450 2900 50  0001 C CNN
+F 1 "+3V3" H 10465 3223 50  0000 C CNN
+F 2 "" H 10450 3050 50  0001 C CNN
+F 3 "" H 10450 3050 50  0001 C CNN
+	1    10450 3050
+	1    0    0    -1
+$EndComp
+Wire Wire Line
+	10450 3150 10450 3050
+NoConn ~ 7800 2850
+NoConn ~ 7800 2950
+$Comp
+L power:GND #PWR0104
+U 1 1 5C8218F5
+P 4300 5800
+F 0 "#PWR0104" H 4300 5550 50  0001 C CNN
+F 1 "GND" H 4300 5650 50  0000 C CNN
+F 2 "" H 4300 5800 50  0000 C CNN
+F 3 "" H 4300 5800 50  0000 C CNN
+	1    4300 5800
+	1    0    0    -1
+$EndComp
+$Comp
+L Connector_Generic:Conn_01x01 J9
+U 1 1 5C8218FB
+P 4300 5300
+F 0 "J9" V 4266 5212 50  0000 R CNN
+F 1 "TP_GND" V 4175 5212 50  0000 R CNN
+F 2 "Connector_PinHeader_2.54mm:PinHeader_1x01_P2.54mm_Vertical" H 4300 5300 50  0001 C CNN
+F 3 "~" H 4300 5300 50  0001 C CNN
+	1    4300 5300
+	0    -1   -1   0
+$EndComp
+Wire Wire Line
+	4300 5500 4300 5800
 $EndSCHEMATC
