File: Hardware/EscaramujoLagoMatch.sch (KiCad schematic (older format))
At the start: 16 parts, among them J1 Jack_3.5mm_5pin, J2 RJ45, U1 MAX662A

Commit message: Add files via upload
Parts:
- removed C7: 1n, Capacitors_ThroughHole:C_Rect_L7_W2.5_P5, symbol C
- removed J1: Jack_3.5mm_5pin, audioJack5Pin:1503_09, symbol Jack_3.5mm_5pin
- removed R1, R3: 51, Resistors_ThroughHole:Resistor_Horizontal_RM7mm, symbol R
- removed RV1: POT, Potentiometers:Potentiometer_Bourns_3296W_3-8Zoll_Inline_ScrewUp, symbol POT
- removed SMA_IN1, SMA_OUT1: SMA_EDGE, sma:SMA, symbol SMA_EDGE
- removed W1, W2: TEST_1P, Measurement_Points:Measurement_Point_Square-TH_Big, symbol TEST_1P
- added C10, C11, C13: 100n, Capacitor_SMD:C_0805_2012Metric_Pad1.15x1.40mm_HandSolder, symbol Device:C
- added C12, C14: 10u, Capacitor_THT:C_Disc_D5.0mm_W2.5mm_P2.50mm, symbol Device:CP
- added C3, C4, C7, C9: 10uF, Capacitor_THT:C_Disc_D5.0mm_W2.5mm_P2.50mm, symbol Device:CP
- added J1: TP_3v3, Connector_PinHeader_2.54mm:PinHeader_1x01_P2.54mm_Vertical, symbol Connector_Generic:Conn_01x01
- added J10: I2C, Connector_PinHeader_2.54mm:PinHeader_1x04_P2.54mm_Vertical, symbol Connector_Generic:Conn_01x04
- added J3: TP_5V, Connector_PinHeader_2.54mm:PinHeader_1x01_P2.54mm_Vertical, symbol Connector_Generic:Conn_01x01
- added J4, J9: TP_GND, Connector_PinHeader_2.54mm:PinHeader_1x01_P2.54mm_Vertical, symbol Connector_Generic:Conn_01x01
- added J5: TEMP_PRES, Connector_PinHeader_2.54mm:PinHeader_1x06_P2.54mm_Vertical, symbol Connector_Generic:Conn_01x06
- added J6: TP_12V, Connector_PinHeader_2.54mm:PinHeader_1x01_P2.54mm_Vertical, symbol Connector_Generic:Conn_01x01
- added J7: RedPitaya, Connector_PinHeader_2.54mm:PinHeader_2x13_P2.54mm_Vertical, symbol Connector_Generic:Conn_02x13_Counter_Clockwise
- added J8: TP_PMT_CTL_V, Connector_PinHeader_2.54mm:PinHeader_1x01_P2.54mm_Vertical, symbol Connector_Generic:Conn_01x01
- added R1: 100k, Resistor_SMD:R_0805_2012Metric_Pad1.15x1.40mm_HandSolder, symbol Device:R
- added R2: 5.1k, Resistor_THT:R_Axial_DIN0207_L6.3mm_D2.5mm_P10.16mm_Horizontal, symbol Device:R
- added R3: 3k, Resistor_THT:R_Axial_DIN0207_L6.3mm_D2.5mm_P10.16mm_Horizontal, symbol Device:R
- added R4, R5: 4k7, Resistor_SMD:R_0805_2012Metric_Pad1.15x1.40mm_HandSolder, symbol Device:R
- added U2: MAX604, Package_DIP:DIP-8_W10.16mm_LongPads, symbol Regulator_Linear:MAX604
- added U3: MAX603, Package_DIP:DIP-8_W10.16mm_LongPads, symbol Regulator_Linear:MAX603
- added U4: TLV5616CD, SOIC127P600X175-8N, symbol TLV5616CD:TLV5616CD
- added U5: LM358, Package_DIP:DIP-8_W10.16mm_LongPads, symbol Amplifier_Operational:LM358
- C1, C2: value 1u -> 2u2; footprint Capacitors_ThroughHole:C_Rect_L7_W2.5_P5 -> Capacitor_THT:C_Disc_D5.0mm_W2.5mm_P2.50mm; symbol CP -> Device:CP
- C5, C6: footprint Capacitors_ThroughHole:C_Rect_L7_W2.5_P5 -> Capacitor_THT:C_Disc_D5.0mm_W2.5mm_P2.50mm; symbol CP -> Device:CP
- C8: footprint Capacitors_ThroughHole:C_Rect_L7_W2.5_P5 -> Capacitor_SMD:C_0805_2012Metric_Pad1.15x1.40mm_HandSolder; symbol C -> Device:C
- J2: footprint Connect:RJ45_8 -> Connector_RJ:RJ45_Amphenol_54602-x08_Horizontal; symbol RJ45 -> EscaramujoLagoMatch-rescue:RJ45
- U1: footprint Housings_DIP:DIP-8_W7.62mm_LongPads -> Package_DIP:DIP-8_W10.16mm_LongPads; symbol MAX662A -> ProjectSpecificParts:MAX662A
Connections:
- net labels added: +3V3, +5V, 5V_UNREG, I2C_SCL, I2C_SDA, PMT_CTRL_V, PMT_CTRL_V_NF, SPI_CLK, SPI_CS, SPI_MOSI
- net labels removed: VCC
- wire segments 58 -> 163
- no-connect marks 8 -> 25
Other:
- moved on the sheet: J2
