File: Hardware/EscaramujoLagoMatch.sch (KiCad schematic (older format))
At the start: 34 parts, among them J1 TP_3v3, J10 I2C, J2 RJ45, J3 TP_5V, J4 TP_GND, J5 TEMP_PRES, J6 TP_12V, J7 RedPitaya, J8 TP_PMT_CTL_V, J9 TP_GND, U1 MAX662A, U2 MAX604, U3 MAX603, U4 TLV5616CD, U5 LM358

Commit message: Add files via upload
Parts:
- removed J5: TEMP_PRES, Connector_PinHeader_2.54mm:PinHeader_1x06_P2.54mm_Vertical, symbol Connector_Generic:Conn_01x06
- removed R5: 4k7, Resistor_SMD:R_0805_2012Metric_Pad1.15x1.40mm_HandSolder, symbol Device:R
- added C15: 100n, Capacitor_SMD:C_0805_2012Metric_Pad1.15x1.40mm_HandSolder, symbol Device:C
- added D1: LED, LED_THT:LED_D5.0mm, symbol Device:LED
- added J5: Sensor, Connector_PinHeader_2.54mm:PinHeader_1x04_P2.54mm_Vertical, symbol Connector_Generic:Conn_01x04
- R4: value 4k7 -> 330; footprint Resistor_SMD:R_0805_2012Metric_Pad1.15x1.40mm_HandSolder -> Resistor_THT:R_Axial_DIN0207_L6.3mm_D2.5mm_P10.16mm_Horizontal
- U1, U2, U3, U5: footprint Package_DIP:DIP-8_W10.16mm_LongPads -> Package_DIP:DIP-8_W7.62mm_Socket
- U4: footprint SOIC127P600X175-8N -> (none)
Connections:
- net +3V3: now also D1.2 (A), J5.1 (Pin_1); no longer R4.1
- net GND: now also J10.2 (Pin_2), R4.2, C15.2, J5.2 (Pin_2); no longer J10.4 (Pin_4)
- net I2C_SCL: now also J5.3 (Pin_3); no longer R4.2
- net I2C_SDA: now also J10.4 (Pin_4), J5.4 (Pin_4); no longer J10.2 (Pin_2)
- net PMT_CTRL_V: now also C15.1
- new net: D1.1 (K), R4.1
- no-connect marks 25 -> 23
Changed lines of the file:
@@
 F 0 "U1" H 2500 4700 60  0000 C CNN
 F 1 "MAX662A" H 2500 4300 60  0000 C CNN
-F 2 "Package_DIP:DIP-8_W10.16mm_LongPads" H 2500 4150 60  0001 C CNN
+F 2 "Package_DIP:DIP-8_W7.62mm_Socket" H 2500 4150 60  0001 C CNN
 F 3 "" H 2500 4150 60  0000 C CNN
 	1    2500 4250
@@
 F 0 "U3" H 3050 1692 50  0000 C CNN
 F 1 "MAX603" H 3050 1601 50  0000 C CNN
-F 2 "Package_DIP:DIP-8_W10.16mm_LongPads" H 3050 1675 50  0001 C CIN
+F 2 "Package_DIP:DIP-8_W7.62mm_Socket" H 3050 1675 50  0001 C CIN
 F 3 "http://datasheets.maximintegrated.com/en/ds/MAX603-MAX604.pdf" H 3050 1300 50  0001 C CNN
 	1    3050 1350
@@
 F 0 "U2" H 3000 3092 50  0000 C CNN
 F 1 "MAX604" H 3000 3001 50  0000 C CNN
-F 2 "Package_DIP:DIP-8_W10.16mm_LongPads" H 3000 3075 50  0001 C CIN
+F 2 "Package_DIP:DIP-8_W7.62mm_Socket" H 3000 3075 50  0001 C CIN
 F 3 "http://datasheets.maximintegrated.com/en/ds/MAX603-MAX604.pdf" H 3000 2700 50  0001 C CNN
 	1    3000 2750
@@
 F 0 "U5" H 9750 4917 50  0000 C CNN
 F 1 "LM358" H 9750 4826 50  0000 C CNN
-F 2 "Package_DIP:DIP-8_W10.16mm_LongPads" H 9750 4550 50  0001 C CNN
+F 2 "Package_DIP:DIP-8_W7.62mm_Socket" H 9750 4550 50  0001 C CNN
 F 3 "http://www.ti.com/lit/ds/symlink/lm2904-n.pdf" H 9750 4550 50  0001 C CNN
 	1    9750 4550
@@
 Text Label 10400 5850 2    50   ~ 0
 PMT_CTRL_V
-$Comp
-L Connector_Generic:Conn_01x06 J5
-U 1 1 5C58EA8E
-P 5950 1600
-F 0 "J5" H 6030 1592 50  0000 L CNN
-F 1 "TEMP_PRES" H 6030 1501 50  0000 L CNN
-F 2 "Connector_PinHeader_2.54mm:PinHeader_1x06_P2.54mm_Vertical" H 5950 1600 50  0001 C CNN
-F 3 "~" H 5950 1600 50  0001 C CNN
-	1    5950 1600
-	1    0    0    -1
-$EndComp
-Wire Wire Line
-	5750 1400 5300 1400
-Wire Wire Line
-	5750 1600 5300 1600
-Text Label 5300 1400 0    50   ~ 0
+Text Label 5500 1650 0    50   ~ 0
 I2C_SCL
-Text Label 5300 1600 0    50   ~ 0
+Text Label 5500 1750 0    50   ~ 0
 I2C_SDA
 $Comp
 L power:+3V3 #PWR012
 U 1 1 5C5A2E81
-P 5100 1800
-F 0 "#PWR012" H 5100 1650 50  0001 C CNN
-F 1 "+3V3" H 5115 1973 50  0000 C CNN
-F 2 "" H 5100 1800 50  0001 C CNN
-F 3 "" H 5100 1800 50  0001 C CNN
-	1    5100 1800
-	1    0    0    -1
-$EndComp
-Wire Wire Line
-	5100 1800 5100 1900
-Wire Wire Line
-	5100 1900 5750 1900
+P 5750 1350
+F 0 "#PWR012" H 5750 1200 50  0001 C CNN
+F 1 "+3V3" H 5765 1523 50  0000 C CNN
+F 2 "" H 5750 1350 50  0001 C CNN
+F 3 "" H 5750 1350 50  0001 C CNN
+	1    5750 1350
+	1    0    0    -1
+$EndComp
 $Comp
 L power:GND #PWR014
 U 1 1 5C5A64E0
-P 5500 2000
-F 0 "#PWR014" H 5500 1750 50  0001 C CNN
-F 1 "GND" H 5505 1827 50  0000 C CNN
-F 2 "" H 5500 2000 50  0001 C CNN
-F 3 "" H 5500 2000 50  0001 C CNN
-	1    5500 2000
-	1    0    0    -1
-$EndComp
-Wire Wire Line
-	5750 1800 5500 1800
-Wire Wire Line
-	5500 1800 5500 2000
-$Comp
-L Device:R R4
-U 1 1 5C5AA499
-P 9350 2750
-F 0 "R4" H 9420 2796 50  0000 L CNN
-F 1 "4k7" H 9420 2705 50  0000 L CNN
-F 2 "Resistor_SMD:R_0805_2012Metric_Pad1.15x1.40mm_HandSolder" V 9280 2750 50  0001 C CNN
-F 3 "~" H 9350 2750 50  0001 C CNN
-	1    9350 2750
-	1    0    0    -1
-$EndComp
-$Comp
-L Device:R R5
-U 1 1 5C5AA4F3
-P 9850 2750
-F 0 "R5" H 9920 2796 50  0000 L CNN
-F 1 "4k7" H 9920 2705 50  0000 L CNN
-F 2 "Resistor_SMD:R_0805_2012Metric_Pad1.15x1.40mm_HandSolder" V 9780 2750 50  0001 C CNN
-F 3 "~" H 9850 2750 50  0001 C CNN
-	1    9850 2750
-	1    0    0    -1
-$EndComp
-$Comp
-L power:+3V3 #PWR021
-U 1 1 5C5AA5B7
-P 9600 2450
-F 0 "#PWR021" H 9600 2300 50  0001 C CNN
-F 1 "+3V3" H 9615 2623 50  0000 C CNN
-F 2 "" H 9600 2450 50  0001 C CNN
-F 3 "" H 9600 2450 50  0001 C CNN
-	1    9600 2450
-	1    0    0    -1
-$EndComp
-Wire Wire Line
-	9850 2600 9850 2500
-Wire Wire Line
-	9850 2500 9600 2500
-Wire Wire Line
-	9600 2500 9600 2450
-Wire Wire Line
-	9350 2600 9350 2500
-Wire Wire Line
-	9350 2500 9600 2500
-Connection ~ 9600 2500
-Wire Wire Line
-	9350 2900 9350 3050
-Wire Wire Line
-	9350 3050 8950 3050
-Text Label 8950 3050 0    50   ~ 0
-I2C_SCL
-Wire Wire Line
-	9850 2900 9850 3050
-Wire Wire Line
-	9850 3050 9450 3050
-Text Label 9450 3050 0    50   ~ 0
-I2C_SDA
+P 5150 1600
+F 0 "#PWR014" H 5150 1350 50  0001 C CNN
+F 1 "GND" H 5155 1427 50  0000 C CNN
+F 2 "" H 5150 1600 50  0001 C CNN
+F 3 "" H 5150 1600 50  0001 C CNN
+	1    5150 1600
+	1    0    0    -1
+$EndComp
 $Comp
 L Connector_Generic:Conn_01x01 J4
@@
 F 0 "U5" H 9350 6217 50  0000 C CNN
 F 1 "LM358" H 9350 6126 50  0000 C CNN
-F 2 "Package_DIP:DIP-8_W10.16mm_LongPads" H 9350 5850 50  0001 C CNN
+F 2 "Package_DIP:DIP-8_W7.62mm_Socket" H 9350 5850 50  0001 C CNN
 F 3 "http://www.ti.com/lit/ds/symlink/lm2904-n.pdf" H 9350 5850 50  0001 C CNN
 	2    9350 5850
@@
 	9750 5850 9650 5850
 Wire Wire Line
-	9750 5850 10400 5850
+	9750 5850 10350 5850
 Connection ~ 9750 5850
 Wire Wire Line
@@
 NoConn ~ 7300 2750
 NoConn ~ 7300 2250
-NoConn ~ 5750 1500
-NoConn ~ 5750 1700
 $Comp
 L power:+5V #PWR0101
@@
 $EndComp
 Wire Wire Line
-	8950 1300 8300 1300
-Wire Wire Line
 	8950 1400 8300 1400
 $Comp
 L power:GND #PWR023
 U 1 1 5C897059
-P 8750 1600
-F 0 "#PWR023" H 8750 1350 50  0001 C CNN
-F 1 "GND" H 8755 1427 50  0000 C CNN
-F 2 "" H 8750 1600 50  0001 C CNN
-F 3 "" H 8750 1600 50  0001 C CNN
-	1    8750 1600
-	1    0    0    -1
-$EndComp
-Wire Wire Line
-	8950 1500 8750 1500
-Wire Wire Line
-	8750 1500 8750 1600
+P 8150 1350
+F 0 "#PWR023" H 8150 1100 50  0001 C CNN
+F 1 "GND" H 8155 1177 50  0000 C CNN
+F 2 "" H 8150 1350 50  0001 C CNN
+F 3 "" H 8150 1350 50  0001 C CNN
+	1    8150 1350
+	1    0    0    -1
+$EndComp
 $Comp
 L power:+3V3 #PWR022
@@
 Wire Wire Line
 	8600 1200 8600 1050
-Text Label 8300 1300 0    50   ~ 0
+Text Label 8300 1500 0    50   ~ 0
 I2C_SDA
 Text Label 8300 1400 0    50   ~ 0
@@
 F 0 "U4" H 8650 5120 50  0000 C CNN
 F 1 "TLV5616CD" H 8650 5029 50  0000 C CNN
-F 2 "SOIC127P600X175-8N" H 8650 4450 50  0001 L BNN
+F 2 "" H 8650 4450 50  0001 L BNN
 F 3 "Texas Instruments" H 8650 4450 50  0001 L BNN
 F 4 "12-Bit, 3 us DAC, Serial Input, Pgrmable Settling Time/Power Consump., Voltage O/P ange=2x V ef. 8-SOIC 0 to 70" H 8650 4450 50  0001 L BNN "Field4"
@@
 F 0 "U5" H 10508 3496 50  0000 L CNN
 F 1 "LM358" H 10508 3405 50  0000 L CNN
-F 2 "Package_DIP:DIP-8_W10.16mm_LongPads" H 10550 3450 50  0001 C CNN
+F 2 "Package_DIP:DIP-8_W7.62mm_Socket" H 10550 3450 50  0001 C CNN
 F 3 "http://www.ti.com/lit/ds/symlink/lm2904-n.pdf" H 10550 3450 50  0001 C CNN
 	3    10550 3450
@@
 	1    0    0    -1
 $EndComp
+$Comp
+L Connector_Generic:Conn_01x04 J5
+U 1 1 5CE05E3E
+P 6100 1550
+F 0 "J5" H 6180 1542 50  0000 L CNN
+F 1 "Sensor" H 6180 1451 50  0000 L CNN
+F 2 "Connector_PinHeader_2.54mm:PinHeader_1x04_P2.54mm_Vertical" H 6100 1550 50  0001 C CNN
+F 3 "~" H 6100 1550 50  0001 C CNN
+	1    6100 1550
+	1    0    0    -1
+$EndComp
+Wire Wire Line
+	5900 1450 5750 1450
+Wire Wire Line
+	5750 1450 5750 1350
+Wire Wire Line
+	5150 1550 5150 1600
+Wire Wire Line
+	5900 1650 5500 1650
+Wire Wire Line
+	5900 1750 5500 1750
+$Comp
+L Device:LED D1
+U 1 1 5CE56B47
+P 7500 1100
+F 0 "D1" H 7491 1316 50  0000 C CNN
+F 1 "LED" H 7491 1225 50  0000 C CNN
+F 2 "LED_THT:LED_D5.0mm" H 7500 1100 50  0001 C CNN
+F 3 "~" H 7500 1100 50  0001 C CNN
+	1    7500 1100
+	0    -1   -1   0
+$EndComp
+$Comp
+L Device:R R4
+U 1 1 5CE5DA89
+P 7500 1450
+F 0 "R4" H 7570 1496 50  0000 L CNN
+F 1 "330" H 7570 1405 50  0000 L CNN
+F 2 "Resistor_THT:R_Axial_DIN0207_L6.3mm_D2.5mm_P10.16mm_Horizontal" V 7430 1450 50  0001 C CNN
+F 3 "~" H 7500 1450 50  0001 C CNN
+	1    7500 1450
+	1    0    0    -1
+$EndComp
+Wire Wire Line
+	5150 1550 5900 1550
+$Comp
+L power:+3V3 #PWR08
+U 1 1 5CE8D132
+P 7500 900
+F 0 "#PWR08" H 7500 750 50  0001 C CNN
+F 1 "+3V3" H 7515 1073 50  0000 C CNN
+F 2 "" H 7500 900 50  0001 C CNN
+F 3 "" H 7500 900 50  0001 C CNN
+	1    7500 900
+	1    0    0    -1
+$EndComp
+$Comp
+L power:GND #PWR09
+U 1 1 5CE8D185
+P 7500 1650
+F 0 "#PWR09" H 7500 1400 50  0001 C CNN
+F 1 "GND" H 7505 1477 50  0000 C CNN
+F 2 "" H 7500 1650 50  0001 C CNN
+F 3 "" H 7500 1650 50  0001 C CNN
+	1    7500 1650
+	1    0    0    -1
+$EndComp
+Wire Wire Line
+	7500 1250 7500 1300
+Wire Wire Line
+	7500 950  7500 900
+Wire Wire Line
+	7500 1600 7500 1650
+Wire Wire Line
+	8950 1500 8300 1500
+Wire Wire Line
+	8950 1300 8150 1300
+Wire Wire Line
+	8150 1300 8150 1350
+$Comp
+L Device:C C15
+U 1 1 5CE4EED1
+P 10350 6100
+F 0 "C15" H 10375 6200 50  0000 L CNN
+F 1 "100n" H 10375 6000 50  0000 L CNN
+F 2 "Capacitor_SMD:C_0805_2012Metric_Pad1.15x1.40mm_HandSolder" H 10388 5950 50  0001 C CNN
+F 3 "" H 10350 6100 50  0000 C CNN
+	1    10350 6100
+	1    0    0    -1
+$EndComp
+Wire Wire Line
+	10350 5950 10350 5850
+Connection ~ 10350 5850
+Wire Wire Line
+	10350 5850 10400 5850
+$Comp
+L power:GND #PWR0105
+U 1 1 5CE71E70
+P 10350 6300
+F 0 "#PWR0105" H 10350 6050 50  0001 C CNN
+F 1 "GND" H 10355 6127 50  0000 C CNN
+F 2 "" H 10350 6300 50  0001 C CNN
+F 3 "" H 10350 6300 50  0001 C CNN
+	1    10350 6300
+	1    0    0    -1
+$EndComp
+Wire Wire Line
+	10350 6300 10350 6250
 $EndSCHEMATC
