File: Hardware/EscaramujoLagoMatch_print.kicad_pcb (KiCad board)
At the start: 2 copper layers, 96 parts, among them J11 Jack_3.5mm_5pin, J11 RJ45, J12 Jack_3.5mm_5pin, J12 RJ45, J21 Jack_3.5mm_5pin, J21 RJ45, J22 Jack_3.5mm_5pin, J22 RJ45, J31 Jack_3.5mm_5pin, J31 RJ45, J32 Jack_3.5mm_5pin, J32 RJ45, U11 MAX662A, U12 MAX662A, U21 MAX662A, U22 MAX662A, U31 MAX662A, U32 MAX662A

Commit message: Add files via upload
Parts:
- removed the C11 at (70.9, 54.7)
- removed the C11 at (70.8, 57.7)
- removed the C11 at (95.3, 60.4)
- removed the C11 at (68.8, 41.0)
- removed the C11 at (57.2, 52.5)
- removed the C11 at (91.8, 57.9)
- removed the C12 at (68.8, 111.0)
- removed the C12 at (70.9, 124.7)
- removed the C12 at (91.8, 127.9)
- removed the C12 at (95.3, 130.4)
- removed the C12 at (70.8, 127.7)
- removed the C12 at (57.2, 122.5)
- removed C21 (x2), C22 (x2), C31 (x2), C32 (x2): 10u, Capacitors_ThroughHole:C_Rect_L7_W2.5_P5
- removed C21 (x2), C22 (x2), C31 (x2), C32 (x2): 1u, Capacitors_ThroughHole:C_Rect_L7_W2.5_P5
- removed C21, C22, C31, C32: 100n, Capacitors_ThroughHole:C_Rect_L7_W2.5_P5
- removed C21, C22, C31, C32: 1n, Capacitors_ThroughHole:C_Rect_L7_W2.5_P5
- removed J11, J12, J21, J22, J31, J32: Jack_3.5mm_5pin, audioJack5Pin:1503_09
- removed J11, J12, J21, J22, J31, J32: RJ45, Connect:RJ45_8
- removed R11 (x2), R12 (x2), R21 (x2), R22 (x2), R31 (x2), R32 (x2): 51, Resistors_ThroughHole:Resistor_Horizontal_RM7mm
- removed RV11, RV12, RV21, RV22, RV31, RV32: POT, Potentiometers:Potentiometer_Bourns_3296W_3-8Zoll_Inline_ScrewUp
- removed SMA_IN11, SMA_IN12, SMA_IN21, SMA_IN22, SMA_IN31, SMA_IN32, SMA_OUT11, SMA_OUT12, SMA_OUT21, SMA_OUT22, SMA_OUT31, SMA_OUT32: SMA_EDGE, sma:SMA
- removed U11, U12, U21, U22, U31, U32: MAX662A, Housings_DIP:DIP-8_W7.62mm_LongPads
- removed W11 (x2), W12 (x2), W21 (x2), W22 (x2), W31 (x2), W32 (x2): TEST_1P, Measurement_Points:Measurement_Point_Square-TH_Big
- added C1: 2u2, Capacitor_THT:C_Disc_D5.0mm_W2.5mm_P2.50mm, F.Cu at (193.0, 48.3)
- added C1: 2u2, Capacitor_THT:C_Disc_D5.0mm_W2.5mm_P2.50mm, F.Cu at (57.1, 142.2)
- added C1: 2u2, Capacitor_THT:C_Disc_D5.0mm_W2.5mm_P2.50mm, F.Cu at (58.4, 49.5)
- added C10: 100n, Capacitor_SMD:C_0805_2012Metric_Pad1.15x1.40mm_HandSolder, B.Cu at (248.9, 29.5)
- added C10: 100n, Capacitor_SMD:C_0805_2012Metric_Pad1.15x1.40mm_HandSolder, B.Cu at (113.0, 123.4)
- added C10: 100n, Capacitor_SMD:C_0805_2012Metric_Pad1.15x1.40mm_HandSolder, B.Cu at (114.3, 30.7)
- added C11: 100n, Capacitor_SMD:C_0805_2012Metric_Pad1.15x1.40mm_HandSolder, B.Cu at (214.6, 28.2)
- added C11: 100n, Capacitor_SMD:C_0805_2012Metric_Pad1.15x1.40mm_HandSolder, B.Cu at (78.7, 122.2)
- added C11: 100n, Capacitor_SMD:C_0805_2012Metric_Pad1.15x1.40mm_HandSolder, B.Cu at (80.0, 29.5)
- added C12: 10u, Capacitor_THT:C_Disc_D5.0mm_W2.5mm_P2.50mm, F.Cu at (232.4, 55.9)
- added C12: 10u, Capacitor_THT:C_Disc_D5.0mm_W2.5mm_P2.50mm, F.Cu at (96.5, 149.9)
- added C12: 10u, Capacitor_THT:C_Disc_D5.0mm_W2.5mm_P2.50mm, F.Cu at (97.8, 57.1)
- added C2: 2u2, Capacitor_THT:C_Disc_D5.0mm_W2.5mm_P2.50mm, F.Cu at (193.0, 50.8)
- added C2: 2u2, Capacitor_THT:C_Disc_D5.0mm_W2.5mm_P2.50mm, F.Cu at (57.1, 144.8)
- added C2: 2u2, Capacitor_THT:C_Disc_D5.0mm_W2.5mm_P2.50mm, F.Cu at (58.4, 52.1)
- added C3: 10uF, Capacitor_THT:C_Disc_D5.0mm_W2.5mm_P2.50mm, F.Cu at (218.4, 38.1)
- added C3: 10uF, Capacitor_THT:C_Disc_D5.0mm_W2.5mm_P2.50mm, F.Cu at (82.5, 132.1)
- added C3: 10uF, Capacitor_THT:C_Disc_D5.0mm_W2.5mm_P2.50mm, F.Cu at (83.8, 39.4)
- added C4: 10uF, Capacitor_THT:C_Disc_D5.0mm_W2.5mm_P2.50mm, F.Cu at (193.0, 35.5)
- added C4: 10uF, Capacitor_THT:C_Disc_D5.0mm_W2.5mm_P2.50mm, F.Cu at (57.1, 129.5)
- added C4: 10uF, Capacitor_THT:C_Disc_D5.0mm_W2.5mm_P2.50mm, F.Cu at (58.4, 36.8)
- added C5: 10u, Capacitor_THT:C_Disc_D5.0mm_W2.5mm_P2.50mm, F.Cu at (229.9, 41.9)
- added C5: 10u, Capacitor_THT:C_Disc_D5.0mm_W2.5mm_P2.50mm, F.Cu at (94.0, 135.9)
- added C5: 10u, Capacitor_THT:C_Disc_D5.0mm_W2.5mm_P2.50mm, F.Cu at (95.3, 43.2)
- added C6: 10u, Capacitor_THT:C_Disc_D5.0mm_W2.5mm_P2.50mm, F.Cu at (213.4, 50.8)
- added C6: 10u, Capacitor_THT:C_Disc_D5.0mm_W2.5mm_P2.50mm, F.Cu at (77.5, 144.7)
- added C6: 10u, Capacitor_THT:C_Disc_D5.0mm_W2.5mm_P2.50mm, F.Cu at (78.7, 52.0)
- added C7: 10uF, Capacitor_THT:C_Disc_D5.0mm_W2.5mm_P2.50mm, F.Cu at (242.6, 28.0)
- added C7: 10uF, Capacitor_THT:C_Disc_D5.0mm_W2.5mm_P2.50mm, F.Cu at (106.7, 122.0)
- added C7: 10uF, Capacitor_THT:C_Disc_D5.0mm_W2.5mm_P2.50mm, F.Cu at (108.0, 29.2)
- added C8: 100n, Capacitor_SMD:C_0805_2012Metric_Pad1.15x1.40mm_HandSolder, B.Cu at (218.4, 49.8)
- added C8: 100n, Capacitor_SMD:C_0805_2012Metric_Pad1.15x1.40mm_HandSolder, B.Cu at (82.5, 143.8)
- added C8: 100n, Capacitor_SMD:C_0805_2012Metric_Pad1.15x1.40mm_HandSolder, B.Cu at (83.8, 51.0)
- added C9: 10uF, Capacitor_THT:C_Disc_D5.0mm_W2.5mm_P2.50mm, F.Cu at (219.7, 26.7)
- added C9: 10uF, Capacitor_THT:C_Disc_D5.0mm_W2.5mm_P2.50mm, F.Cu at (83.8, 120.7)
- added C9: 10uF, Capacitor_THT:C_Disc_D5.0mm_W2.5mm_P2.50mm, F.Cu at (85.1, 28.0)
- added J1: TP_3v3, Connector_PinHeader_2.54mm:PinHeader_1x01_P2.54mm_Vertical, F.Cu at (259.1, 36.8)
- added J1: TP_3v3, Connector_PinHeader_2.54mm:PinHeader_1x01_P2.54mm_Vertical, F.Cu at (123.2, 130.8)
- added J1: TP_3v3, Connector_PinHeader_2.54mm:PinHeader_1x01_P2.54mm_Vertical, F.Cu at (124.5, 38.1)
- added J10: I2C, Connector_PinHeader_2.54mm:PinHeader_1x04_P2.54mm_Vertical, F.Cu at (219.7, 82.8)
- added J10: I2C, Connector_PinHeader_2.54mm:PinHeader_1x04_P2.54mm_Vertical, F.Cu at (83.8, 176.8)
- added J10: I2C, Connector_PinHeader_2.54mm:PinHeader_1x04_P2.54mm_Vertical, F.Cu at (85.1, 84.1)
- added J2: RJ45, Connector_RJ:RJ45_Amphenol_54602-x08_Horizontal, F.Cu at (252.7, 53.3)
- added J2: RJ45, Connector_RJ:RJ45_Amphenol_54602-x08_Horizontal, F.Cu at (116.8, 147.3)
- added J2: RJ45, Connector_RJ:RJ45_Amphenol_54602-x08_Horizontal, F.Cu at (118.1, 54.6)
- added J3: TP_5V, Connector_PinHeader_2.54mm:PinHeader_1x01_P2.54mm_Vertical, F.Cu at (252.7, 36.8)
- added J3: TP_5V, Connector_PinHeader_2.54mm:PinHeader_1x01_P2.54mm_Vertical, F.Cu at (116.8, 130.8)
- added J3: TP_5V, Connector_PinHeader_2.54mm:PinHeader_1x01_P2.54mm_Vertical, F.Cu at (118.1, 38.1)
- added J4: TP_GND, Connector_PinHeader_2.54mm:PinHeader_1x01_P2.54mm_Vertical, F.Cu at (265.4, 36.8)
- added J4: TP_GND, Connector_PinHeader_2.54mm:PinHeader_1x01_P2.54mm_Vertical, F.Cu at (129.5, 130.8)
- added J4: TP_GND, Connector_PinHeader_2.54mm:PinHeader_1x01_P2.54mm_Vertical, F.Cu at (130.8, 38.1)
- added J5: TEMP_PRES, Connector_PinHeader_2.54mm:PinHeader_1x06_P2.54mm_Vertical, F.Cu at (229.4, 74.7)
- added J5: TEMP_PRES, Connector_PinHeader_2.54mm:PinHeader_1x06_P2.54mm_Vertical, F.Cu at (93.5, 168.7)
- added J5: TEMP_PRES, Connector_PinHeader_2.54mm:PinHeader_1x06_P2.54mm_Vertical, F.Cu at (94.7, 75.9)
- added J6: TP_12V, Connector_PinHeader_2.54mm:PinHeader_1x01_P2.54mm_Vertical, F.Cu at (246.4, 36.8)
- added J6: TP_12V, Connector_PinHeader_2.54mm:PinHeader_1x01_P2.54mm_Vertical, F.Cu at (110.5, 130.8)
- added J6: TP_12V, Connector_PinHeader_2.54mm:PinHeader_1x01_P2.54mm_Vertical, F.Cu at (111.8, 38.1)
- added J7: RedPitaya, Connector_PinHeader_2.54mm:PinHeader_2x13_P2.54mm_Vertical, F.Cu at (177.8, 30.5)
- added J7: RedPitaya, Connector_PinHeader_2.54mm:PinHeader_2x13_P2.54mm_Vertical, F.Cu at (41.9, 124.5)
- added J7: RedPitaya, Connector_PinHeader_2.54mm:PinHeader_2x13_P2.54mm_Vertical, F.Cu at (43.2, 31.8)
- added J8: TP_PMT_CTL_V, Connector_PinHeader_2.54mm:PinHeader_1x01_P2.54mm_Vertical, F.Cu at (251.5, 64.8)
- added J8: TP_PMT_CTL_V, Connector_PinHeader_2.54mm:PinHeader_1x01_P2.54mm_Vertical, F.Cu at (115.6, 158.8)
- added J8: TP_PMT_CTL_V, Connector_PinHeader_2.54mm:PinHeader_1x01_P2.54mm_Vertical, F.Cu at (116.8, 66.0)
- added J9: TP_GND, Connector_PinHeader_2.54mm:PinHeader_1x01_P2.54mm_Vertical, F.Cu at (251.5, 72.4)
- added J9: TP_GND, Connector_PinHeader_2.54mm:PinHeader_1x01_P2.54mm_Vertical, F.Cu at (115.6, 166.4)
- added J9: TP_GND, Connector_PinHeader_2.54mm:PinHeader_1x01_P2.54mm_Vertical, F.Cu at (116.8, 73.7)
- added R1: 100k, Resistor_SMD:R_0805_2012Metric_Pad1.15x1.40mm_HandSolder, B.Cu at (231.1, 61.2)
- added R1: 100k, Resistor_SMD:R_0805_2012Metric_Pad1.15x1.40mm_HandSolder, B.Cu at (95.2, 155.2)
- added R1: 100k, Resistor_SMD:R_0805_2012Metric_Pad1.15x1.40mm_HandSolder, B.Cu at (96.5, 62.5)
- added R2: 15k, Resistor_THT:R_Axial_DIN0207_L6.3mm_D2.5mm_P10.16mm_Horizontal, F.Cu at (232.4, 50.8)
- added R2: 15k, Resistor_THT:R_Axial_DIN0207_L6.3mm_D2.5mm_P10.16mm_Horizontal, F.Cu at (96.5, 144.8)
- added R2: 15k, Resistor_THT:R_Axial_DIN0207_L6.3mm_D2.5mm_P10.16mm_Horizontal, F.Cu at (97.8, 52.1)
- added R3: 18k, Resistor_THT:R_Axial_DIN0207_L6.3mm_D2.5mm_P10.16mm_Horizontal, F.Cu at (215.6, 55.9)
- added R3: 18k, Resistor_THT:R_Axial_DIN0207_L6.3mm_D2.5mm_P10.16mm_Horizontal, F.Cu at (79.8, 149.9)
- added R3: 18k, Resistor_THT:R_Axial_DIN0207_L6.3mm_D2.5mm_P10.16mm_Horizontal, F.Cu at (81.0, 57.1)
- added R4: 4k7, Resistor_SMD:R_0805_2012Metric_Pad1.15x1.40mm_HandSolder, B.Cu at (224.3, 87.4)
- added R4: 4k7, Resistor_SMD:R_0805_2012Metric_Pad1.15x1.40mm_HandSolder, B.Cu at (88.4, 181.4)
- added R4: 4k7, Resistor_SMD:R_0805_2012Metric_Pad1.15x1.40mm_HandSolder, B.Cu at (89.7, 88.7)
- added R5: 4k7, Resistor_SMD:R_0805_2012Metric_Pad1.15x1.40mm_HandSolder, B.Cu at (221.7, 87.4)
- added R5: 4k7, Resistor_SMD:R_0805_2012Metric_Pad1.15x1.40mm_HandSolder, B.Cu at (85.9, 181.4)
- added R5: 4k7, Resistor_SMD:R_0805_2012Metric_Pad1.15x1.40mm_HandSolder, B.Cu at (87.1, 88.7)
- added U1: MAX662A, Package_DIP:DIP-8_W10.16mm_LongPads, F.Cu at (198.1, 45.7)
- added U1: MAX662A, Package_DIP:DIP-8_W10.16mm_LongPads, F.Cu at (62.2, 139.7)
- added U1: MAX662A, Package_DIP:DIP-8_W10.16mm_LongPads, F.Cu at (63.5, 47.0)
- added U2: MAX604, Package_DIP:DIP-8_W10.16mm_LongPads, F.Cu at (226.1, 27.9)
- added U2: MAX604, Package_DIP:DIP-8_W10.16mm_LongPads, F.Cu at (90.2, 121.9)
- added U2: MAX604, Package_DIP:DIP-8_W10.16mm_LongPads, F.Cu at (91.4, 29.2)
- added U3: MAX603, Package_DIP:DIP-8_W10.16mm_LongPads, F.Cu at (198.1, 27.9)
- added U3: MAX603, Package_DIP:DIP-8_W10.16mm_LongPads, F.Cu at (62.2, 121.9)
- added U3: MAX603, Package_DIP:DIP-8_W10.16mm_LongPads, F.Cu at (63.5, 29.2)
- added U4: MCP41100, Package_DIP:DIP-8_W10.16mm_LongPads, F.Cu at (198.1, 61.0)
- added U4: MCP41100, Package_DIP:DIP-8_W10.16mm_LongPads, F.Cu at (62.2, 154.9)
- added U4: MCP41100, Package_DIP:DIP-8_W10.16mm_LongPads, F.Cu at (63.5, 62.2)
- added U5: LM358, Package_DIP:DIP-8_W10.16mm_LongPads, F.Cu at (234.9, 62.2)
- added U5: LM358, Package_DIP:DIP-8_W10.16mm_LongPads, F.Cu at (99.1, 156.2)
- added U5: LM358, Package_DIP:DIP-8_W10.16mm_LongPads, F.Cu at (100.3, 63.5)
Routing:
- net (no net): track 0.00 -> 1244.3 mm, vias 0 -> 18
- net GND: track 1434.8 -> 737.8 mm, vias 12 -> 4
- net VCC: track 582.7 -> 0.00 mm
- net +3V3: track 0.00 -> 467.7 mm, vias 0 -> 12
- net +5V: track 0.00 -> 240.0 mm, vias 0 -> 4
- net Net-(J2-Pad3): track 183.5 -> 0.00 mm
- net /I2C_SDA: track 0.00 -> 176.5 mm
- net /12V: track 284.2 -> 114.5 mm, vias 0 -> 4
- net /I2C_SCL: track 0.00 -> 160.9 mm, vias 0 -> 4
- net Net-(R1-Pad1): track 135.0 -> 0.00 mm
- net /5V_UNREG: track 0.00 -> 128.4 mm, vias 0 -> 4
- net Net-(C7-Pad2): track 114.0 -> 0.00 mm
- net /PMT_CTRL_V: track 0.00 -> 88.0 mm
- net /SPI_CS: track 0.00 -> 85.5 mm, vias 0 -> 4
- net Net-(R3-Pad2): track 0.00 -> 61.5 mm
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- added copper zone on B.Cu, net (none)
Other:
- board outline added: 248.9 x 174 mm
- net class Default: trace_width 0.4 -> 0.75; via_dia 1.4 -> 2
- board text added: "12V"
- board text added: "3v3"
- board text added: "5V"
- board text added: "GND"
- board text added: "Vctrl PMT"
- board text removed: "+5 VDC"
- board text removed: "LAGO + Escaramujo"
- board text removed: "OUT"
- board text removed: "PMT IN"
